File: Hardware/SparkFun_Thing_Plus_ESP32_WROOM_C.sch (EAGLE design)
At the start: 58 parts, among them J2 MICRO-SDFRICTION, J3 QWIIC_RA, J5 THING_PLUS_LOGICAL, Q2 MBT3904DW1T1, Q3 20V/4.2A/52mΩ/1.4W, U1 MCP73831, U2 ESP-WROOM-3232D-NARROW, U3 XC6222B331MR-G, U4 MAX17048, U5 XC6222B331MR-G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

Commit message: Update BOM for cap mismatch.
Accidentally placed C4/C5 in the wrong spot. Made the change in schematic so no board reorder is necessary.
Parts:
- C4: value 0.1uF -> 10uF; device SparkFun-Capacitors:0.1UF-0402T-6.3V-10%-X7R -> SparkFun-Capacitors:10UF-0402T-6.3V-20%
- C5: value 10uF -> 0.1uF; device SparkFun-Capacitors:10UF-0402T-6.3V-20% -> SparkFun-Capacitors:0.1UF-0402T-6.3V-10%-X7R
Other:
- moved on the sheet: C4, C5
Changed lines of the file:
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@@
 <setting verticaltext="up"/>
 </settings>
-<grid distance="0.1" unitdist="inch" unit="inch" style="lines" multiple="1" display="yes" altdistance="0.01" altunitdist="inch" altunit="inch"/>
+<grid distance="0.1" unitdist="inch" unit="inch" style="lines" multiple="1" display="no" altdistance="0.01" altunitdist="inch" altunit="inch"/>
 <layers>
 <layer number="1" name="Top" color="4" fill="1" visible="no" active="no"/>
@@
 <part name="SUPPLY15" library="SparkFun-PowerSymbols" deviceset="3.3V" device=""/>
 <part name="GND10" library="SparkFun-PowerSymbols" deviceset="GND" device=""/>
-<part name="C4" library="SparkFun-Capacitors" deviceset="0.1UF" device="-0402T-6.3V-10%-X7R" value="0.1uF"/>
+<part name="C4" library="SparkFun-Capacitors" deviceset="10UF" device="-0402T-6.3V-20%" value="10uF"/>
 <part name="SUPPLY16" library="SparkFun-PowerSymbols" deviceset="3.3V" device=""/>
 <part name="GND37" library="SparkFun-PowerSymbols" deviceset="GND" device=""/>
@@
 <part name="SUPPLY20" library="SparkFun-PowerSymbols" deviceset="3.3V" device=""/>
 <part name="GND12" library="SparkFun-PowerSymbols" deviceset="GND" device=""/>
-<part name="C5" library="SparkFun-Capacitors" deviceset="10UF" device="-0402T-6.3V-20%" value="10uF"/>
+<part name="C5" library="SparkFun-Capacitors" deviceset="0.1UF" device="-0402T-6.3V-10%-X7R" value="0.1uF"/>
 <part name="SUPPLY21" library="SparkFun-PowerSymbols" deviceset="3.3V" device=""/>
 <part name="GND13" library="SparkFun-PowerSymbols" deviceset="GND" device=""/>
@@
 <attribute name="VALUE" x="304.8" y="154.686" size="1.778" layer="96" align="top-center"/>
 </instance>
-<instance part="C4" gate="G$1" x="327.66" y="162.56" smashed="yes">
-<attribute name="NAME" x="329.184" y="165.481" size="1.778" layer="95" font="vector"/>
-<attribute name="VALUE" x="329.184" y="160.401" size="1.778" layer="96" font="vector"/>
-</instance>
-<instance part="SUPPLY16" gate="G$1" x="327.66" y="170.18" smashed="yes">
-<attribute name="VALUE" x="327.66" y="172.974" size="1.778" layer="96" align="bottom-center"/>
-</instance>
-<instance part="GND37" gate="1" x="327.66" y="154.94" smashed="yes">
-<attribute name="VALUE" x="327.66" y="154.686" size="1.778" layer="96" align="top-center"/>
+<instance part="C4" gate="G$1" x="76.2" y="30.48" smashed="yes">
+<attribute name="NAME" x="77.724" y="33.401" size="1.778" layer="95" font="vector"/>
+<attribute name="VALUE" x="77.724" y="28.321" size="1.778" layer="96" font="vector"/>
+</instance>
+<instance part="SUPPLY16" gate="G$1" x="76.2" y="38.1" smashed="yes">
+<attribute name="VALUE" x="76.2" y="40.894" size="1.778" layer="96" align="bottom-center"/>
+</instance>
+<instance part="GND37" gate="1" x="76.2" y="22.86" smashed="yes">
+<attribute name="VALUE" x="76.2" y="22.606" size="1.778" layer="96" align="top-center"/>
 </instance>
 <instance part="D5" gate="G$1" x="304.8" y="165.1" smashed="yes">
@@
 <attribute name="VALUE" x="48.26" y="14.986" size="1.778" layer="96" align="top-center"/>
 </instance>
-<instance part="C5" gate="G$1" x="76.2" y="30.48" smashed="yes">
-<attribute name="NAME" x="77.724" y="33.401" size="1.778" layer="95" font="vector"/>
-<attribute name="VALUE" x="77.724" y="28.321" size="1.778" layer="96" font="vector"/>
-</instance>
-<instance part="SUPPLY21" gate="G$1" x="76.2" y="38.1" smashed="yes">
-<attribute name="VALUE" x="76.2" y="40.894" size="1.778" layer="96" align="bottom-center"/>
-</instance>
-<instance part="GND13" gate="1" x="76.2" y="22.86" smashed="yes">
-<attribute name="VALUE" x="76.2" y="22.606" size="1.778" layer="96" align="top-center"/>
+<instance part="C5" gate="G$1" x="327.66" y="162.56" smashed="yes">
+<attribute name="NAME" x="329.184" y="165.481" size="1.778" layer="95" font="vector"/>
+<attribute name="VALUE" x="329.184" y="160.401" size="1.778" layer="96" font="vector"/>
+</instance>
+<instance part="SUPPLY21" gate="G$1" x="327.66" y="170.18" smashed="yes">
+<attribute name="VALUE" x="327.66" y="172.974" size="1.778" layer="96" align="bottom-center"/>
+</instance>
+<instance part="GND13" gate="1" x="327.66" y="154.94" smashed="yes">
+<attribute name="VALUE" x="327.66" y="154.686" size="1.778" layer="96" align="top-center"/>
 </instance>
 <instance part="J4" gate="G$1" x="205.74" y="243.84" smashed="yes" rot="MR90">
@@
 <pinref part="C4" gate="G$1" pin="1"/>
 <pinref part="SUPPLY16" gate="G$1" pin="3.3V"/>
-<wire x1="327.66" y1="170.18" x2="327.66" y2="167.64" width="0.1524" layer="91"/>
+<wire x1="76.2" y1="38.1" x2="76.2" y2="35.56" width="0.1524" layer="91"/>
 </segment>
 <segment>
@@
 <pinref part="SUPPLY21" gate="G$1" pin="3.3V"/>
 <pinref part="C5" gate="G$1" pin="1"/>
-<wire x1="76.2" y1="38.1" x2="76.2" y2="35.56" width="0.1524" layer="91"/>
+<wire x1="327.66" y1="170.18" x2="327.66" y2="167.64" width="0.1524" layer="91"/>
 </segment>
 <segment>
@@
 <pinref part="C4" gate="G$1" pin="2"/>
 <pinref part="GND37" gate="1" pin="GND"/>
-<wire x1="327.66" y1="160.02" x2="327.66" y2="157.48" width="0.1524" layer="91" style="longdash"/>
+<wire x1="76.2" y1="27.94" x2="76.2" y2="25.4" width="0.1524" layer="91" style="longdash"/>
 </segment>
 <segment>
@@
 <pinref part="C5" gate="G$1" pin="2"/>
 <pinref part="GND13" gate="1" pin="GND"/>
-<wire x1="76.2" y1="27.94" x2="76.2" y2="25.4" width="0.1524" layer="91"/>
-</segment>
-<segment>
+<wire x1="327.66" y1="160.02" x2="327.66" y2="157.48" width="0.1524" layer="91"/>
+</segment>
+<segment>

Commit message: Swap VREG IC
Parts:
- U3, U5: value XC6222B331MR-G -> 3.3V; device SparkFun-IC-Power:XC6222B331MR-G -> SparkFun-IC-Power:V_REG_AP2112K-3.3V
Other:
- note added: "600mA out"
- note added: "600mA out 6V max in"
- note removed: "700mA out"
- note removed: "700mA out 6V max in"
Changed lines of the file:
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@@
 <part name="LOGO1" library="SparkFun-Aesthetics" deviceset="SFE_LOGO_NAME_FLAME" device=".1_INCH" value="SFE_LOGO_NAME_FLAME.1_INCH"/>
 <part name="JP2" library="SparkFun-Jumpers" deviceset="JUMPER-SMT_2_NC_TRACE" device="_SILK" package3d_urn="urn:adsk.eagle:package:39281/1" value="JUMPER-SMT_2_NC_TRACE_SILK"/>
-<part name="U3" library="SparkFun-IC-Power" deviceset="XC6222" device="B331MR-G"/>
-<part name="U5" library="SparkFun-IC-Power" deviceset="XC6222" device="B331MR-G"/>
+<part name="U3" library="SparkFun-IC-Power" deviceset="V_REG_AP2112" device="K-3.3V" value="3.3V"/>
+<part name="U5" library="SparkFun-IC-Power" deviceset="V_REG_AP2112" device="K-3.3V" value="3.3V"/>
 <part name="J2" library="SparkFun-Connectors" deviceset="MICRO-SD" device="FRICTION"/>
 <part name="U2" library="SparkFun-RF" deviceset="ESP-WROOM-32" device="32D-NARROW"/>
@@
 <text x="60.96" y="271.78" size="2.54" layer="94" font="vector" align="center">System Regulator</text>
 <text x="167.64" y="266.7" size="2.54" layer="94" font="vector" align="center">Lithium-Polymer Battery Charger</text>
-<text x="68.58" y="226.06" size="1.778" layer="97" font="vector" align="top-center">700mA out
+<text x="68.58" y="226.06" size="1.778" layer="97" font="vector" align="top-center">600mA out
 6V max in</text>
 <text x="60.96" y="190.5" size="2.54" layer="94" font="vector" align="center">Auto-Reset</text>
@@
 <wire x1="345.44" y1="279.4" x2="345.44" y2="203.2" width="0.2032" layer="97" style="longdash"/>
 <wire x1="269.24" y1="134.62" x2="340.36" y2="134.62" width="0.2032" layer="97" style="longdash"/>
-<text x="175.26" y="17.78" size="1.778" layer="97" font="vector" align="center">700mA out</text>
+<text x="175.26" y="17.78" size="1.778" layer="97" font="vector" align="center">600mA out</text>
 <text x="307.34" y="187.96" size="2.54" layer="94" font="vector" align="center">RGB Status LED</text>
 <text x="58.42" y="55.88" size="2.54" layer="94" font="vector" align="center">microSD Connector</text>
